File: sfp-snoop.kicad_pcb (KiCad board)
At the start: 2 copper layers, 22.9 x 53.3 mm, 29 parts, among them J1 SFP+, J2 Conn_01x20, J3 Conn_01x20, U1 AIC1221-33GY3TR, U2 AP2191WG-7

Commit message: GPIO23 jumper
Parts:
- moved C4 0.21 mm to (144.0, 67.8)
- moved R10 0.06 mm to (144.6, 72.0)
Routing:
- net /GPIO23: track 7.96 -> 6.76 mm
